File: Fonte/fonte.brd (EAGLE design)
At the start: 100 x 80 mm, 14 parts, among them T1 BC337

Commit message: substituindo arquivos eagle
Parts:
- C1: device rcl:PANASONIC_D -> rcl:E5-10,5
- R1: value 750 -> 1k
- moved R1 59.9 mm to (29.2, 38.1), turned to 0 degrees
- moved T1 58.9 mm to (48.3, 74.9), turned to 0 degrees
- moved R3 51.1 mm to (91.4, 39.4), turned to 270 degrees
- moved R4 24.4 mm to (49.5, 10.2), turned to 0 degrees
- moved LED1 24.1 mm to (41.9, 27.9), turned to 270 degrees
- moved D2 21.9 mm to (29.2, 61.0)
- moved D4 20.4 mm to (27.9, 50.8), turned to 0 degrees
- moved D5 18.9 mm to (29.2, 26.7), turned to 0 degrees
- moved D3 16.6 mm to (7.62, 50.8), turned to 180 degrees
- moved C1 15.7 mm to (14.0, 26.7), turned to 0 degrees
- moved D1 15.7 mm to (7.62, 61.0), turned to 0 degrees
- moved R2 12.0 mm to (17.8, 40.6)
- moved VOUT 10.9 mm to (91.4, 71.1), turned to 90 degrees
- moved VIN 9.25 mm to (19.1, 76.2), turned to 180 degrees
Routing:
- net N$1: track 0.00 -> 292.3 mm
- net N$2: track 0.00 -> 185.0 mm
- net N$9: track 0.00 -> 67.0 mm
- net N$7: track 0.00 -> 46.2 mm
- net N$4: track 0.00 -> 45.7 mm
- net N$8: track 0.00 -> 44.4 mm
- net N$5: track 0.00 -> 40.6 mm
- net N$3: track 0.00 -> 34.7 mm
- net N$6: track 0.00 -> 30.7 mm
