File: Fonte/fonte.sch (EAGLE design)
At the start: 14 parts, among them T1 BC337

Commit message: substituindo arquivos eagle
Parts:
- C1: device rcl:CPOL-EUD -> rcl:CPOL-EUE5-10.5
- R1: value 750 -> 1k
Other:
- moved on the sheet: C1
Changed lines of the file:
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@@
 <part name="D3" library="diode" library_urn="urn:adsk.eagle:library:210" deviceset="1N4004" device="" package3d_urn="urn:adsk.eagle:package:43336/1"/>
 <part name="D4" library="diode" library_urn="urn:adsk.eagle:library:210" deviceset="1N4004" device="" package3d_urn="urn:adsk.eagle:package:43336/1"/>
-<part name="C1" library="rcl" library_urn="urn:adsk.eagle:library:334" deviceset="CPOL-EU" device="D" package3d_urn="urn:adsk.eagle:package:23424/2" value="680uF"/>
-<part name="R1" library="rcl" library_urn="urn:adsk.eagle:library:334" deviceset="R-EU_" device="0207/10" package3d_urn="urn:adsk.eagle:package:23491/2" value="750"/>
+<part name="R1" library="rcl" library_urn="urn:adsk.eagle:library:334" deviceset="R-EU_" device="0207/10" package3d_urn="urn:adsk.eagle:package:23491/2" value="1k"/>
 <part name="R2" library="rcl" library_urn="urn:adsk.eagle:library:334" deviceset="R-EU_" device="0207/10" package3d_urn="urn:adsk.eagle:package:23491/2" value="2k2"/>
 <part name="R3" library="rcl" library_urn="urn:adsk.eagle:library:334" deviceset="R-EU_" device="0207/10" package3d_urn="urn:adsk.eagle:package:23491/2" value="2k"/>
@@
 <part name="T1" library="transistor" library_urn="urn:adsk.eagle:library:402" deviceset="BC337" device="" package3d_urn="urn:adsk.eagle:package:28523/2"/>
 <part name="D5" library="diode" library_urn="urn:adsk.eagle:library:210" deviceset="1N4728" device="" package3d_urn="urn:adsk.eagle:package:43341/1"/>
+<part name="C1" library="rcl" library_urn="urn:adsk.eagle:library:334" deviceset="CPOL-EU" device="E5-10.5" package3d_urn="urn:adsk.eagle:package:23372/2" value="680uF"/>
 </parts>
 <sheets>
@@
 <attribute name="VALUE" x="22.6314" y="73.66" size="1.778" layer="96" rot="R90"/>
 </instance>
-<instance part="C1" gate="G$1" x="38.1" y="78.74" smashed="yes">
-<attribute name="NAME" x="39.243" y="79.2226" size="1.778" layer="95"/>
-<attribute name="VALUE" x="39.243" y="74.1426" size="1.778" layer="96"/>
-</instance>
 <instance part="R1" gate="G$1" x="60.96" y="91.44" smashed="yes" rot="R90">
 <attribute name="NAME" x="59.4614" y="87.63" size="1.778" layer="95" rot="R90"/>
@@
 <attribute name="VALUE" x="64.389" y="66.802" size="1.778" layer="96" rot="R90"/>
 </instance>
+<instance part="C1" gate="G$1" x="38.1" y="83.82" smashed="yes">
+<attribute name="NAME" x="39.243" y="84.3026" size="1.778" layer="95"/>
+<attribute name="VALUE" x="39.243" y="79.2226" size="1.778" layer="96"/>
+</instance>
 </instances>
 <busses>
@@
 <wire x1="5.08" y1="76.2" x2="5.08" y2="60.96" width="0.1524" layer="91"/>
 <wire x1="5.08" y1="60.96" x2="38.1" y2="60.96" width="0.1524" layer="91"/>
-<pinref part="C1" gate="G$1" pin="-"/>
-<wire x1="38.1" y1="60.96" x2="38.1" y2="73.66" width="0.1524" layer="91"/>
+<wire x1="38.1" y1="60.96" x2="38.1" y2="78.74" width="0.1524" layer="91"/>
 <pinref part="LED1" gate="G$1" pin="C"/>
 <wire x1="38.1" y1="60.96" x2="50.8" y2="60.96" width="0.1524" layer="91"/>
@@
 <wire x1="60.96" y1="66.04" x2="60.96" y2="60.96" width="0.1524" layer="91"/>
 <wire x1="76.2" y1="63.5" x2="76.2" y2="60.96" width="0.1524" layer="91"/>
+<pinref part="C1" gate="G$1" pin="-"/>
 </segment>
 </net>
@@
 <wire x1="25.4" y1="76.2" x2="25.4" y2="96.52" width="0.1524" layer="91"/>
 <junction x="20.32" y="76.2"/>
-<pinref part="C1" gate="G$1" pin="+"/>
+<pinref part="R2" gate="G$1" pin="2"/>
 <wire x1="25.4" y1="96.52" x2="38.1" y2="96.52" width="0.1524" layer="91"/>
-<wire x1="38.1" y1="96.52" x2="38.1" y2="81.28" width="0.1524" layer="91"/>
-<pinref part="R2" gate="G$1" pin="2"/>
 <wire x1="38.1" y1="96.52" x2="50.8" y2="96.52" width="0.1524" layer="91"/>
 <wire x1="50.8" y1="96.52" x2="50.8" y2="86.36" width="0.1524" layer="91"/>
-<junction x="38.1" y="96.52"/>
 <pinref part="R1" gate="G$1" pin="2"/>
 <wire x1="50.8" y1="96.52" x2="60.96" y2="96.52" width="0.1524" layer="91"/>
@@
 <wire x1="88.9" y1="96.52" x2="88.9" y2="91.44" width="0.1524" layer="91"/>
 <junction x="60.96" y="96.52"/>
+<pinref part="C1" gate="G$1" pin="+"/>
+<wire x1="38.1" y1="86.36" x2="38.1" y2="96.52" width="0.1524" layer="91"/>
+<junction x="38.1" y="96.52"/>
 </segment>
 </net>
